Commit message: updatet urdf and tested on real robot

File: source/packages/modulo_core/tests/fixtures/iiwa7.urdf (robot description, URDF)
Before this commit: robot iiwa7, 10 links, 9 joints
Links:
- link iiwa_link_ee: mass 1e-6 -> 1.32
Joints:
- joint iiwa_joint_ee: origin xyz=0 0 0.045 rpy=0 0 0 -> xyz=0 0 0.245 rpy=0 0 0
